File: pcb/divine-light.kicad_pcb (KiCad board)
At the start: 2 copper layers, 0 parts

Commit message: add neopixel sheet, finished battery and main circuitry
Signed-off-by: Toby Cm <toby@vsus.app>
Parts:
- added C1: 100n, Capacitor_SMD:C_0603_1608Metric, F.Cu at (36.0, 34.6)
- added C4: 10u, Capacitor_SMD:C_0603_1608Metric, F.Cu at (43.9, 9.78)
- added C5: 100n, Capacitor_SMD:C_0603_1608Metric, F.Cu at (36.0, 37.1)
- added C6: 100n, Capacitor_SMD:C_0603_1608Metric, F.Cu at (36.0, 39.6)
- added C7: 22u, Capacitor_SMD:C_0805_2012Metric, F.Cu at (52.0, 44.5)
- added C8: 22u, Capacitor_SMD:C_0805_2012Metric, F.Cu at (52.0, 47.5)
- added C9: 10u, Capacitor_SMD:C_0603_1608Metric, F.Cu at (36.0, 42.1)
- added D1: 5V, Diode_SMD:D_SOD-523, F.Cu at (43.8, 25.2)
- added D10: SK6812, LED_SMD:LED_SK6812_PLCC4_5.0x5.0mm_P3.2mm, F.Cu at (120.0, 63.3)
- added D11: SK6812, LED_SMD:LED_SK6812_PLCC4_5.0x5.0mm_P3.2mm, F.Cu at (140.0, 73.3)
- added D12: SK6812, LED_SMD:LED_SK6812_PLCC4_5.0x5.0mm_P3.2mm, F.Cu at (140.0, 93.3)
- added D13: SK6812, LED_SMD:LED_SK6812_PLCC4_5.0x5.0mm_P3.2mm, F.Cu at (170.0, 63.3)
- added D14: SK6812, LED_SMD:LED_SK6812_PLCC4_5.0x5.0mm_P3.2mm, F.Cu at (120.0, 73.3)
- added D15: SK6812, LED_SMD:LED_SK6812_PLCC4_5.0x5.0mm_P3.2mm, F.Cu at (150.0, 63.3)
- added D16: SK6812, LED_SMD:LED_SK6812_PLCC4_5.0x5.0mm_P3.2mm, F.Cu at (110.0, 83.3)
- added D17: SK6812, LED_SMD:LED_SK6812_PLCC4_5.0x5.0mm_P3.2mm, F.Cu at (150.0, 73.3)
- added D18: SK6812, LED_SMD:LED_SK6812_PLCC4_5.0x5.0mm_P3.2mm, F.Cu at (160.0, 93.3)
- added D19: SK6812, LED_SMD:LED_SK6812_PLCC4_5.0x5.0mm_P3.2mm, F.Cu at (170.0, 83.3)
- added D2: SK6812, LED_SMD:LED_SK6812_PLCC4_5.0x5.0mm_P3.2mm, F.Cu at (130.0, 93.3)
- added D20: SK6812, LED_SMD:LED_SK6812_PLCC4_5.0x5.0mm_P3.2mm, F.Cu at (110.0, 93.3)
- added D21: SK6812, LED_SMD:LED_SK6812_PLCC4_5.0x5.0mm_P3.2mm, F.Cu at (120.0, 83.3)
- added D22: SK6812, LED_SMD:LED_SK6812_PLCC4_5.0x5.0mm_P3.2mm, F.Cu at (150.0, 93.3)
- added D23: SK6812, LED_SMD:LED_SK6812_PLCC4_5.0x5.0mm_P3.2mm, F.Cu at (130.0, 63.3)
- added D24: SK6812, LED_SMD:LED_SK6812_PLCC4_5.0x5.0mm_P3.2mm, F.Cu at (110.0, 63.3)
- added D25: SK6812, LED_SMD:LED_SK6812_PLCC4_5.0x5.0mm_P3.2mm, F.Cu at (160.0, 73.3)
- added D26: SK6812, LED_SMD:LED_SK6812_PLCC4_5.0x5.0mm_P3.2mm, F.Cu at (170.0, 93.3)
- added D27: SK6812, LED_SMD:LED_SK6812_PLCC4_5.0x5.0mm_P3.2mm, F.Cu at (180.0, 63.3)
- added D28: SK6812, LED_SMD:LED_SK6812_PLCC4_5.0x5.0mm_P3.2mm, F.Cu at (150.0, 83.3)
- added D29: SK6812, LED_SMD:LED_SK6812_PLCC4_5.0x5.0mm_P3.2mm, F.Cu at (140.0, 63.3)
- added D3: SK6812, LED_SMD:LED_SK6812_PLCC4_5.0x5.0mm_P3.2mm, F.Cu at (130.0, 73.3)
- added D30: SK6812, LED_SMD:LED_SK6812_PLCC4_5.0x5.0mm_P3.2mm, F.Cu at (160.0, 63.3)
- added D31: SK6812, LED_SMD:LED_SK6812_PLCC4_5.0x5.0mm_P3.2mm, F.Cu at (130.0, 83.3)
- added D32: SK6812, LED_SMD:LED_SK6812_PLCC4_5.0x5.0mm_P3.2mm, F.Cu at (110.0, 73.3)
- added D33: SK6812, LED_SMD:LED_SK6812_PLCC4_5.0x5.0mm_P3.2mm, F.Cu at (160.0, 83.3)
- added D4: SK6812, LED_SMD:LED_SK6812_PLCC4_5.0x5.0mm_P3.2mm, F.Cu at (170.0, 73.3)
- added D5: SK6812, LED_SMD:LED_SK6812_PLCC4_5.0x5.0mm_P3.2mm, F.Cu at (140.0, 83.3)
- added D6: SK6812, LED_SMD:LED_SK6812_PLCC4_5.0x5.0mm_P3.2mm, F.Cu at (180.0, 93.3)
- added D7: SK6812, LED_SMD:LED_SK6812_PLCC4_5.0x5.0mm_P3.2mm, F.Cu at (120.0, 93.3)
- added D8: SK6812, LED_SMD:LED_SK6812_PLCC4_5.0x5.0mm_P3.2mm, F.Cu at (180.0, 73.3)
- added D9: SK6812, LED_SMD:LED_SK6812_PLCC4_5.0x5.0mm_P3.2mm, F.Cu at (180.0, 83.3)
- added F1: 2A, Fuse:Fuse_1206_3216Metric, F.Cu at (44.7, 17.7)
- added FB1: 220Ω@100MHz, Resistor_SMD:R_0805_2012Metric_Pad1.20x1.40mm_HandSolder, F.Cu at (49.5, 20.8)
- added H1: MountingHole, MountingHole:MountingHole_3.2mm_M3_Pad, F.Cu at (105.0, 55.0)
- added H2: MountingHole, MountingHole:MountingHole_3.2mm_M3_Pad, F.Cu at (185.0, 55.0)
- added H3: MountingHole, MountingHole:MountingHole_3.2mm_M3_Pad, F.Cu at (105.0, 100.0)
- added H4: MountingHole, MountingHole:MountingHole_3.2mm_M3_Pad, F.Cu at (185.0, 100.0)
- added J1: Battery_JST, Connector_JST:JST_PH_S2B-PH-K_1x02_P2.00mm_Horizontal, F.Cu at (46.1, 35.7)
- added J2: Battery_JST, Connector_JST:JST_PH_S2B-PH-K_1x02_P2.00mm_Horizontal, F.Cu at (54.1, 35.7)
- added J3: USB_C_Receptacle_USB2.0_14P, easyeda2kicad:USB-C-SMD_TYPE-C-16PIN-2MD-073, F.Cu at (47.4, 2.93)
- added Q1: FS8205A, Package_TO_SOT_SMD:SOT-23-6, F.Cu at (40.6, 35.7)
- added R1: 330, Resistor_SMD:R_0603_1608Metric, F.Cu at (36.0, 44.6)
- added R2: 2k, Resistor_SMD:R_0805_2012Metric, F.Cu at (56.5, 44.4)
- added R3: 5.1k, Resistor_SMD:R_0603_1608Metric, F.Cu at (43.9, 12.3)
- added R4: 5.1k, Resistor_SMD:R_0603_1608Metric, F.Cu at (43.9, 14.8)
- added R5: 330, Resistor_SMD:R_0603_1608Metric, F.Cu at (36.0, 47.1)
- added U1: IP2326, Package_DFN_QFN:VQFN-24-1EP_4x4mm_P0.5mm_EP2.5x2.5mm, F.Cu at (46.7, 46.1)
- added U2: HY2120CB, Package_TO_SOT_SMD:SOT-23-6, F.Cu at (40.6, 40.3)
- added U3: CH572D, Package_DFN_QFN:QFN-20-1EP_3x3mm_P0.4mm_EP1.65x1.65mm, F.Cu at (49.0, 11.2)
- added U4: USBLC6-2SC6, Package_TO_SOT_SMD:SOT-23-6, F.Cu at (44.5, 21.8)
- added U5: TPS54308, Package_TO_SOT_SMD:SOT-23-6, F.Cu at (40.6, 45.0)
Other:
- board outline added: 90 x 55 mm

Commit message: initial pcb routing done
Signed-off-by: Toby Cm <toby@vsus.app>
Parts:
- added AE2: Antenna_Shield, wch-antenna:ANT-F-1-2.4G-1.6MM-FR4-WCH, F.Cu at (171.0, 101.0)
- added C10: 22u, Capacitor_SMD:C_0805_2012Metric, F.Cu at (132.5, 52.0)
- added C11: 22u, Capacitor_SMD:C_0805_2012Metric, F.Cu at (146.0, 53.2)
- added C12: C, Capacitor_SMD:C_0603_1608Metric, F.Cu at (155.0, 98.0)
- added C13: C, Capacitor_SMD:C_0603_1608Metric, F.Cu at (160.0, 98.0)
- added C14: 22u, Capacitor_SMD:C_0805_2012Metric, F.Cu at (123.8, 58.8)
- added C2: 100n, Capacitor_SMD:C_0603_1608Metric, F.Cu at (131.5, 57.8)
- added C3: 8p, Capacitor_SMD:C_0603_1608Metric, F.Cu at (152.5, 103.5)
- added F2: 1A, Fuse:Fuse_0805_2012Metric, F.Cu at (180.0, 88.0)
- added FB2: 220Ω@100MHz, Resistor_SMD:R_0805_2012Metric_Pad1.20x1.40mm_HandSolder, F.Cu at (175.8, 88.0)
- added J4: USB_C_Receptacle_USB2.0_14P, easyeda2kicad:USB-C-SMD_TYPE-C-16PIN-2MD-073, F.Cu at (133.0, 100.0)
- added J5: USB_C_Receptacle_USB2.0_14P, easyeda2kicad:USB-C-SMD_TYPE-C-16PIN-2MD-073, F.Cu at (187.4, 88.0)
- added L1: 2.2u, Inductor_SMD:L_APV_APH0630, F.Cu at (153.0, 55.0)
- added L2: 2.2u, Inductor_SMD:L_APV_APH0630, F.Cu at (140.0, 55.0)
- added L3: L, Inductor_SMD:L_0603_1608Metric, F.Cu at (157.5, 97.2)
- added R10: 5.1k, Resistor_SMD:R_0603_1608Metric, F.Cu at (140.0, 101.0)
- added R11: 56k, Resistor_SMD:R_0603_1608Metric, F.Cu at (187.8, 94.2)
- added R12: 56k, Resistor_SMD:R_0603_1608Metric, F.Cu at (187.8, 81.8)
- added R13: 82k, Resistor_SMD:R_0603_1608Metric, F.Cu at (147.0, 77.8)
- added R14: 330, Resistor_SMD:R_0603_1608Metric, F.Cu at (169.9, 57.0)
- added R6: 10k, Resistor_SMD:R_0603_1608Metric, F.Cu at (133.5, 59.5)
- added R7: 56k, Resistor_SMD:R_0603_1608Metric, F.Cu at (129.5, 59.5)
- added R8: 90k, Resistor_SMD:R_1206_3216Metric, B.Cu at (160.0, 52.0)
- added R9: 5.1k, Resistor_SMD:R_0603_1608Metric, F.Cu at (126.0, 101.0)
- added TH1: 100k @ 3950K, Resistor_SMD:R_0603_1608Metric, B.Cu at (145.0, 77.8)
- added U6: SS12D10G6-WJ, easyeda2kicad:SW-TH_3P-P4.80_HX-SS12D10G6-WJ, F.Cu at (115.5, 58.8)
- added Y1: 32Mhz, Crystal:Crystal_SMD_2016-4Pin_2.0x1.6mm, F.Cu at (152.5, 101.2)
- C4: value 10u -> 8p
- C9: value 10u -> 22u; footprint Capacitor_SMD:C_0603_1608Metric -> Capacitor_SMD:C_0805_2012Metric
- D1: value 5V -> LED; footprint Diode_SMD:D_SOD-523 -> LED_SMD:LED_0603_1608Metric
- H4: footprint MountingHole:MountingHole_3.2mm_M3_Pad -> MountingHole:MountingHole_3.2mm_M3
- J1, J2: moved to B.Cu
- moved R3 156.7 mm to (187.8, 74.5), turned to 180 degrees
- moved J3 154.4 mm to (187.4, 68.0), turned to 90 degrees
- moved R4 151.2 mm to (187.8, 61.5), turned to 180 degrees
- moved C6 145.2 mm to (180.5, 54.0), turned to 90 degrees
- moved C5 145.0 mm to (180.2, 51.5)
- moved R5 144.9 mm to (180.5, 57.5), turned to 90 degrees
- moved C4 143.9 mm to (155.0, 101.2), turned to -90 degrees
- moved U4 143.2 mm to (180.0, 68.2), turned to 180 degrees
- moved R1 141.2 mm to (177.0, 51.5)
- moved U2 137.1 mm to (177.0, 54.2)
- moved F1 135.9 mm to (171.0, 68.0), turned to 180 degrees
- moved D1 133.6 mm to (173.5, 57.0), turned to 180 degrees
- moved U3 133.2 mm to (148.5, 99.8), turned to 180 degrees
- moved Q1 132.7 mm to (172.0, 54.2)
- moved FB1 126.2 mm to (166.5, 68.0), turned to 180 degrees
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Connections:
- net /D+ renamed /BD+
- net /D- renamed /BD-
- C4 pad 1: VBUS -> Net-(U3-XI)
- D1 pad 1: Net-(D1-A1) -> GND
- D1 pad 2: GND -> Net-(D1-A)
- D19 pad 2: Net-(D19-DIN) -> Net-(D18-DOUT)
- D20 pad 2: Net-(D18-DOUT) -> Net-(D19-DOUT)
- D21 pad 2: Net-(D19-DOUT) -> Net-(D20-DOUT)
- D22 pad 2: Net-(D20-DOUT) -> Net-(D21-DOUT)
- D23 pad 2: Net-(D21-DOUT) -> Net-(D22-DOUT)
- D24 pad 2: Net-(D22-DOUT) -> Net-(D23-DOUT)
- D25 pad 2: Net-(D23-DOUT) -> Net-(D24-DOUT)
- D26 pad 2: Net-(D24-DOUT) -> Net-(D25-DOUT)
- D27 pad 2: Net-(D25-DOUT) -> Net-(D26-DOUT)
- D28 pad 2: Net-(D26-DOUT) -> Net-(D27-DOUT)
- D29 pad 2: Net-(D27-DOUT) -> Net-(D28-DOUT)
- D30 pad 2: Net-(D28-DOUT) -> Net-(D29-DOUT)
- D31 pad 2: Net-(D29-DOUT) -> Net-(D30-DOUT)
- D32 pad 2: Net-(D30-DOUT) -> Net-(D31-DOUT)
- D32 pad 4: Net-(D19-DIN) -> Net-(D32-DOUT)
- D33 pad 2: Net-(D31-DOUT) -> Net-(D32-DOUT)
- F1 pad 2: Net-(D1-A1) -> Net-(F1-Pad2)
- FB1 pad 1: Net-(D1-A1) -> Net-(F1-Pad2)
- J1 pad 2: +BATT -> Net-(J1-Pin_2)
- U1 pad 11: unconnected-(U1-ISET-Pad11) -> Net-(U1-ISET)
- U1 pad 4: unconnected-(U1-NTC-Pad4) -> Net-(U1-NTC)
- U1 pad 5: unconnected-(U1-BAT_STAT-Pad5) -> /Battery/STAT
- U1 pad 6: unconnected-(U1-LED-Pad6) -> Net-(U1-LED)
- U3 pad 1: unconnected-(U3-PA3/T/R1/SCL2/SCK_/PWM3/CP0-Pad1) -> /TX
- U3 pad 11: unconnected-(U3-PA0/UDM/R2/T3/SCL1-Pad11) -> /MD-
- U3 pad 12: unconnected-(U3-PA1/UDP/R3/T2/SDA1-Pad12) -> /MD+
- U3 pad 13: unconnected-(U3-PA4/SCS/PWM4/TMR2-Pad13) -> /Neopixel/DIN
- U3 pad 14: unconnected-(U3-PA5/SCK/SCL3-Pad14) -> /Battery/STAT
- U3 pad 19: Net-(U3-NC-Pad19) -> unconnected-(U3-NC-Pad19)_1
- U3 pad 2: unconnected-(U3-XO-Pad2) -> Net-(U3-XO)
- U3 pad 20: unconnected-(U3-PA2/R/T1/SDA2/SCS_/PWM2/TMR1/CN-Pad20) -> /RX
- U3 pad 3: unconnected-(U3-XI-Pad3) -> Net-(U3-XI)
- U3 pad 4: Net-(U3-NC-Pad19) -> unconnected-(U3-NC-Pad19)
- U3 pad 5: unconnected-(U3-ANT-Pad5) -> /ANT
- U3 pad 6: unconnected-(U3-VDD33-Pad6) -> +3V3
- U3 pad 7: unconnected-(U3-VIO33-Pad7) -> +3V3
- U3 pad 8: unconnected-(U3-V5-Pad8) -> +5V
- U5 pad 2: unconnected-(U5-SW-Pad2) -> Net-(U5-SW)
- U5 pad 3: unconnected-(U5-VIN-Pad3) -> +BATT
- U5 pad 4: unconnected-(U5-FB-Pad4) -> Net-(U5-FB)
- U5 pad 5: unconnected-(U5-EN-Pad5) -> /Battery/EN
- U5 pad 6: unconnected-(U5-BOOT-Pad6) -> Net-(U5-BOOT)
Routing:
- net +5V: track 0.00 -> 389.4 mm, vias 0 -> 3
- net /Battery/STAT: track 0.00 -> 147.2 mm, vias 0 -> 4
- net Net-(D17-DOUT): track 0.00 -> 84.9 mm, vias 0 -> 2
- net Net-(D10-DIN): track 0.00 -> 80.6 mm, vias 0 -> 4
- net Net-(D25-DOUT): track 0.00 -> 80.4 mm, vias 0 -> 2
- net /Neopixel/DIN: track 0.00 -> 73.5 mm, vias 0 -> 2
- net +BATT: track 0.00 -> 69.3 mm, vias 0 -> 3
- net /Battery/VC: track 0.00 -> 61.7 mm, vias 0 -> 2
- net Net-(U1-NTC): track 0.00 -> 49.0 mm, vias 0 -> 6
- net VBUS: track 0.00 -> 41.6 mm, vias 0 -> 3
- net /BD+: track 0.00 -> 33.0 mm
- net /BD-: track 0.00 -> 32.9 mm
- net -BATT: track 0.00 -> 19.2 mm, vias 0 -> 1
- net /MD-: track 0.00 -> 18.9 mm
- net /MD+: track 0.00 -> 18.8 mm
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- added copper zone on F.Cu, net +BATT
- added copper zone on B.Cu, net GND
- added copper zone on F.Cu, net GND
- added copper zone on F.Cu, net Net-(C1-Pad1)
- added copper zone on F.Cu, net Net-(U5-SW)
