File: pcb/divine-light.kicad_sch (KiCad schematic)
At the start: 9 parts, among them J3 USB_C_Receptacle_USB2.0_14P, U3 CH552E, U4 USBLC6-2SC6

Commit message: add neopixel sheet, finished battery and main circuitry
Signed-off-by: Toby Cm <toby@vsus.app>
Parts:
- removed D1: 5V, Diode_SMD:D_SOD-523, symbol Device:D_TVS
- removed U3: CH552E, easyeda2kicad:MSOP-10_L3.0-W3.0-P0.50-LS5.0-BL, symbol easyeda2kicad:CH552E
- added C3: 8p, Capacitor_SMD:C_0603_1608Metric, symbol Device:C
- added F2: 1A, Fuse:Fuse_0805_2012Metric, symbol Device:Polyfuse
- added FB2: 220Ω@100MHz, Resistor_SMD:R_0805_2012Metric_Pad1.20x1.40mm_HandSolder, symbol Device:FerriteBead
- added H1, H2, H3, H4: MountingHole, MountingHole:MountingHole_3.2mm_M3_Pad, symbol Mechanical:MountingHole
- added J4, J5: USB_C_Receptacle_USB2.0_14P, easyeda2kicad:USB-C-SMD_TYPE-C-16PIN-2MD-073, symbol Connector:USB_C_Receptacle_USB2.0_14P
- added R10, R9: 5.1k, Resistor_SMD:R_0603_1608Metric, symbol Device:R
- added R11, R12: 56k, Resistor_SMD:R_0603_1608Metric, symbol Device:R
- added U3: CH572D, Package_DFN_QFN:QFN-20-1EP_3x3mm_P0.4mm_EP1.65x1.65mm, symbol easyeda2kicad:CH572D
- added Y1: 32Mhz, Crystal:Crystal_SMD_2016-4Pin_2.0x1.6mm, symbol Device:Crystal_GND24
- C4: value 10u -> 8p; LCSC Part C96446 -> C327316
Connections:
- net D+: no longer J3.A6 (D+), J3.B6 (D+)
- net D-: no longer J3.A7 (D-), J3.B7 (D-)
- net GND: now also C3.2, J4.A1 (GND), J4.A12 (GND), J4.B1 (GND), J4.B12 (GND), J4.SH (SHIELD), J5.A1 (GND), J5.A12 (GND), J5.B1 (GND), J5.B12 (GND), J5.SH (SHIELD), R10.2, R11.2, R12.2, R9.2, U3.21 (GND), Y1.2 (G), Y1.4 (G)
- net VBUS: no longer C4.1
- new net: J5.A5 (CC1), R11.1
- new net: C3.1, U3.2 (XO), Y1.1
- new net: J4.A5 (CC1), R9.1
- new net: F2.1, J5.A4 (VBUS), J5.A9 (VBUS), J5.B4 (VBUS), J5.B9 (VBUS)
- new net: J5.B5 (CC2), R12.1
- new net: C4.1, U3.3 (XI), Y1.3
- new net: J4.B5 (CC2), R10.1
- new net: J4.A4 (VBUS), J4.A9 (VBUS), J4.B4 (VBUS), J4.B9 (VBUS)
- new net: F2.2, FB2.1
- new net: U3.19 (NC), U3.4 (NC)
- new net +3V3: U3.6 (VDD33), U3.7 (VIO33)
- new net +5V: FB2.2, U3.8 (V5)
- new net ANT: U3.5 (ANT)
- new net BD+: J3.A6 (D+), J3.B6 (D+)
- new net BD-: J3.A7 (D-), J3.B7 (D-)
- new net Battery/STAT: U3.14 (PA5/SCK/SCL3)
- new net MD+: J4.A6 (D+), J4.B6 (D+), U3.12 (PA1/UDP/R3/T2/SDA1)
- new net MD-: J4.A7 (D-), J4.B7 (D-), U3.11 (PA0/UDM/R2/T3/SCL1)
- new net Neopixel/DIN: U3.13 (PA4/SCS/PWM4/TMR2)
- new net RX: U3.20 (PA2/R/T1/SDA2/SCS_/PWM2/TMR1/CN)
- new net TX: U3.1 (PA3/T/R1/SCL2/SCK_/PWM3/CP0)
- no-connect marks 0 -> 10
Other:
- added sheet Neopixel (neopixel.kicad_sch)
- sheet Battery ports: added EN, STAT; removed none

Commit message: initial pcb routing done
Signed-off-by: Toby Cm <toby@vsus.app>
Parts:
- added AE2: Antenna_Shield, wch-antenna:ANT-F-1-2.4G-1.6MM-FR4-WCH, symbol Device:Antenna_Shield
- added C12, C13: C, Capacitor_SMD:C_0603_1608Metric, symbol Device:C
- added L3: L, Inductor_SMD:L_0603_1608Metric, symbol Device:L
- H4: footprint MountingHole:MountingHole_3.2mm_M3_Pad -> MountingHole:MountingHole_3.2mm_M3
Connections:
- net D+ is gone; now on net BD+: U4.3 (I/O2), U4.4 (I/O2)
- net D- is gone; now on net BD-: U4.1 (I/O1), U4.6 (I/O1)
- net ANT: now also C12.1, L3.1
- net GND: now also AE2.2 (Shield), C12.2, C13.2
- new net: AE2.1 (A), C13.1, L3.2
- no-connect marks 10 -> 13
Other:
- note added: "Charging USB"
- note added: "MCU"
- note added: "MCU USB"
- note added: "Mounting holes"
- note added: "Power bank USB"
- moved on the sheet: C3, C4, F2, FB2, H1, H2, H3, H4, J4, J5, R10, R11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
