File: pcb/neopixel.kicad_sch (KiCad schematic)
At the start: 32 parts

Commit message: initial pcb routing done
Signed-off-by: Toby Cm <toby@vsus.app>
Parts:
- renumbered D20 to D19, D22 to D20, D24 to D21, D26 to D22, D28 to D23, D30 to D24, D32 to D25, D19 to D26, D21 to D27, D23 to D28, D25 to D29, D27 to D30, D29 to D31, D31 to D32
Connections:
- no-connect marks 0 -> 1
